Commit message: Corrected robot description (one motor was 180 degrees wrong) and adjusted joint limits

File: model/robot.urdf (robot description, URDF)
Before this commit: robot leap, 17 links, 16 joints
Joints:
- joint index_dip_joint: limit lower=-0.366 upper=2.042 effort=0.95 velocity=8.48 -> lower=-1.65806 upper=1.867502 effort=0.95 velocity=8.48
- joint index_mcp_joint: limit lower=-0.506 upper=1.885 effort=0.95 velocity=8.48 -> lower=-0.45379 upper=1.570796 effort=0.95 velocity=8.48
- joint index_pip_abb_joint: limit lower=-1.047 upper=1.047 effort=0.95 velocity=8.48 -> lower=-1.378810 upper=1.378810 effort=0.95 velocity=8.48
- joint index_pip_flex_joint: limit lower=-0.314 upper=2.23 effort=0.95 velocity=8.48 -> lower=-0.31416 upper=2.3038 effort=0.95 velocity=8.48
- joint middle_dip_joint: limit lower=-0.366 upper=2.042 effort=0.95 velocity=8.48 -> lower=-1.65806 upper=1.867502 effort=0.95 velocity=8.48
- joint middle_mcp_joint: limit lower=-0.506 upper=1.885 effort=0.95 velocity=8.48 -> lower=-0.45379 upper=1.570796 effort=0.95 velocity=8.48
- joint middle_pip_abb_joint: limit lower=-1.047 upper=1.047 effort=0.95 velocity=8.48 -> lower=-1.378810 upper=1.378810 effort=0.95 velocity=8.48
- joint middle_pip_flex_joint: limit lower=-0.314 upper=2.23 effort=0.95 velocity=8.48 -> lower=-0.31416 upper=2.3038 effort=0.95 velocity=8.48
- joint ring_dip_joint: limit lower=-0.366 upper=2.042 effort=0.95 velocity=8.48 -> lower=-1.65806 upper=1.867502 effort=0.95 velocity=8.48
- joint ring_mcp_joint: limit lower=-0.506 upper=1.885 effort=0.95 velocity=8.48 -> lower=-0.45379 upper=1.570796 effort=0.95 velocity=8.48
- joint ring_pip_abb_joint: limit lower=-1.047 upper=1.047 effort=0.95 velocity=8.48 -> lower=-1.378810 upper=1.378810 effort=0.95 velocity=8.48
- joint ring_pip_flex_joint: limit lower=-0.314 upper=2.23 effort=0.95 velocity=8.48 -> lower=-0.31416 upper=2.3038 effort=0.95 velocity=8.48
- joint thumb_cmc_abb_joint: limit lower=-0.349 upper=2.094 effort=0.95 velocity=8.48 -> lower=-0.38397 upper=2.02458 effort=0.95 velocity=8.48
- joint thumb_cmc_flex_joint: limit lower=-2.47 upper=2.443 effort=0.95 velocity=8.48 -> lower=-0.7854 upper=1.570796 effort=0.95 velocity=8.48; origin xyz=0 0.0143 -0.013 rpy=1.5707963267948958919 1.5707963267948958919 0 -> xyz=0 0.0143 -0.013 rpy=1.5707963267948958919 -1.5707963267948958919 0
- joint thumb_ip_joint: limit lower=-1.34 upper=1.88 effort=0.95 velocity=8.48 -> lower=-0.7854 upper=1.93731 effort=0.95 velocity=8.48
- joint thumb_mcp_joint: limit lower=-1.20 upper=1.90 effort=0.95 velocity=8.48 -> lower=-0.34906 upper=1.7453 effort=0.95 velocity=8.48
